File: pcb/theseus/bgkeeb.kicad_sch (KiCad schematic)
At the start: 104 parts, among them J1 Pimoroni, SW1 SW_Push, SW11 SW_Push, SW12 SW_Push, SW13 SW_Push, SW14 SW_Push, SW15 SW_Push, SW2 SW_Push, SW21 SW_Push, SW22 SW_Push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

Commit message: Bye Promicro, Hello RP2040-Zero (with Xiao compatibility... almost!)
Parts:
- removed U1: ProMicro, Keebio-Parts:ArduinoProMicro, symbol keebio:ProMicro
- added J2: Bat+ pth, Connector_PinSocket_2.54mm:PinSocket_1x01_P2.54mm_Vertical, symbol Connector:Conn_01x01_Socket
- added J3: reset pth, Connector_PinSocket_2.54mm:PinSocket_1x01_P2.54mm_Vertical, symbol Connector:Conn_01x01_Socket
- added J4: rp2040-zero-tht-bottom-bodged, Connector_PinSocket_2.54mm:PinSocket_1x05_P2.54mm_Vertical, symbol Connector:Conn_01x05_Socket
- added J5: ~, fingerpunch:vik-connector-horizontal, symbol theseus:vik-keyboard-connector-fix
- added JP1: SolderJumper_3_Bridged12, Jumper:SolderJumper-3_P1.3mm_Bridged12_Pad1.0x1.5mm_NumberLabels, symbol Jumper:SolderJumper_3_Bridged12
- added U1: rp2040-zero-tht-sides, theseus:rp2040-zero-tht-nocut, symbol theseus:rp2040-zero
Connections:
- net +5V: now also J5.6 (5V), JP1.1 (A), U1.23 (5V); no longer U3.4 (RING2), U4.4 (RING2)
- net ENC1A: now also U1.8 (7)
- net ENC1B: now also U1.9 (8)
- net GND: now also J5.2 (GND), J5.7 (GND), U1.22 (GND)
- net RESET: now also J3.1 (Pin_1)
- net col0: now also U1.20 (29)
- net col1: now also U1.19 (28)
- net col2: now also U1.18 (27)
- net col3: now also U1.17 (26)
- net col4: now also U1.2 (1)
- net data: now also U1.7 (6)
- net led: now also U1.1 (0)
- net row0: now also U1.3 (2)
- net row1: now also U1.4 (3)
- net row2: now also U1.5 (4)
- net row3: now also U1.6 (5)
- net scl: now also J5.4 (SCL), U1.16 (15)
- net sda: now also J5.3 (SDA), U1.15 (14)
- net raw renamed Bat+ Pad
- net Bat+ Pad: now also J2.1 (Pin_1)
- new net: JP1.2 (C), U3.4 (RING2), U4.4 (RING2)
- new net +3.3V: J5.1 (3V3), JP1.3 (B), U1.21 (3V3)
- new net CS: J4.1 (Pin_14), J5.10 (SPI_CS)
- new net GPIO_X1: J4.5 (Pin_10), J5.9 (GPIO_AD)
- new net SCK: J4.4 (Pin_11), J5.12 (SCLK)
- new net SPI RX: J4.2 (Pin_13), J5.11 (MISO)
- new net SPI TX: J4.3 (Pin_12), J5.8 (MOSI)
- no-connect marks 3 -> 5
Other:
- note added: "VIK OUT"
- moved on the sheet: BATJ2, U3, U4
